File: PCB/temp4c.kicad_pcb (KiCad board)
At the start: 2 copper layers, 98 x 50 mm, 38 parts, among them J1 Probes, J2 Probes, J3 eflashy32, J4 24VAC, J5 USB_C_Receptacle_USB2.0, U1 ESP32-WROOM-32D, U2 BD9G101G, U3 AMS1117-3.3

Commit message: fix ground pin on eflashy32
Parts:
- moved J3 12.7 mm to (121.0, 46.4), turned to 0 degrees
Connections:
- J3 pad 1: /GPIO0 -> GND
- J3 pad 2: /EN -> /TXD
- J3 pad 3: 3V3 -> /RXD
- J3 pad 4: /RXD -> 3V3
- J3 pad 5: /TXD -> /EN
- J3 pad 6: GND -> /GPIO0
Changed lines of the file:
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@@
   (net 40 "unconnected-(U1-Pad36)")
   (net 41 "unconnected-(U1-Pad37)")
-  (net 42 "Net-(J4-Pad2)")
-  (net 43 "Net-(J4-Pad1)")
+  (net 42 "Net-(D1-Pad1)")
+  (net 43 "Net-(F1-Pad1)")
   (net 44 "PROBE_BUS")
   (net 45 "Net-(J5-PadA5)")
@@
     (fp_line (start -2.25 -1.6) (end 2.25 -1.6) (layer "F.Fab") (width 0.1))
     (pad "1" smd roundrect (at -2.1375 0 270) (size 1.125 3.4) (layers "F.Cu" "F.Paste" "F.Mask") (roundrect_rratio 0.222222)
-      (net 43 "Net-(J4-Pad1)") (pintype "passive"))
+      (net 43 "Net-(F1-Pad1)") (pintype "passive"))
     (pad "2" smd roundrect (at 2.1375 0 270) (size 1.125 3.4) (layers "F.Cu" "F.Paste" "F.Mask") (roundrect_rratio 0.222222)
       (net 7 "Net-(D3-Pad1)") (pintype "passive"))
@@
     (fp_circle (center 5.08 0) (end 6.58 0) (layer "F.Fab") (width 0.1) (fill none))
     (pad "1" thru_hole rect (at 0 0 180) (size 2.6 2.6) (drill 1.3) (layers F&B.Cu *.Mask)
-      (net 43 "Net-(J4-Pad1)") (pinfunction "Pin_1") (pintype "passive"))
+      (net 43 "Net-(F1-Pad1)") (pinfunction "Pin_1") (pintype "passive"))
     (pad "2" thru_hole circle (at 5.08 0 180) (size 2.6 2.6) (drill 1.3) (layers F&B.Cu *.Mask)
-      (net 42 "Net-(J4-Pad2)") (pinfunction "Pin_2") (pintype "passive"))
+      (net 42 "Net-(D1-Pad1)") (pinfunction "Pin_2") (pintype "passive"))
     (model "${KICAD6_3DMODEL_DIR}/TerminalBlock_Phoenix.3dshapes/TerminalBlock_Phoenix_MKDS-1,5-2-5.08_1x02_P5.08mm_Horizontal.wrl"
       (offset (xyz 0 0 0))
@@
   )
   (footprint "Connector_PinHeader_2.54mm:PinHeader_1x06_P2.54mm_Vertical" (layer "F.Cu")
-    (at 121 59.12 180)
+    (at 121 46.42)
     (descr "Through hole straight pin header, 1x06, 2.54mm pitch, single row")
     (tags "Through hole pin header THT 1x06 2.54mm single row")
@@
     (fp_line (start 1.27 -1.27) (end 1.27 13.97) (layer "F.Fab") (width 0.1))
     (fp_line (start 1.27 13.97) (end -1.27 13.97) (layer "F.Fab") (width 0.1))
-    (pad "1" thru_hole rect (at 0 0 180) (size 1.7 1.7) (drill 1) (layers *.Cu *.Mask)
-      (net 2 "/GPIO0") (pinfunction "Pin_1") (pintype "passive"))
-    (pad "2" thru_hole oval (at 0 2.54 180) (size 1.7 1.7) (drill 1) (layers *.Cu *.Mask)
-      (net 3 "/EN") (pinfunction "Pin_2") (pintype "passive"))
-    (pad "3" thru_hole oval (at 0 5.08 180) (size 1.7 1.7) (drill 1) (layers *.Cu *.Mask)
-      (net 8 "3V3") (pinfunction "Pin_3") (pintype "passive"))
-    (pad "4" thru_hole oval (at 0 7.62 180) (size 1.7 1.7) (drill 1) (layers *.Cu *.Mask)
-      (net 4 "/RXD") (pinfunction "Pin_4") (pintype "passive"))
-    (pad "5" thru_hole oval (at 0 10.16 180) (size 1.7 1.7) (drill 1) (layers *.Cu *.Mask)
-      (net 5 "/TXD") (pinfunction "Pin_5") (pintype "passive"))
-    (pad "6" thru_hole oval (at 0 12.7 180) (size 1.7 1.7) (drill 1) (layers *.Cu *.Mask)
-      (net 1 "GND") (pinfunction "Pin_6") (pintype "passive"))
+    (pad "1" thru_hole rect (at 0 0) (size 1.7 1.7) (drill 1) (layers *.Cu *.Mask)
+      (net 1 "GND") (pinfunction "Pin_1") (pintype "passive"))
+    (pad "2" thru_hole oval (at 0 2.54) (size 1.7 1.7) (drill 1) (layers *.Cu *.Mask)
+      (net 5 "/TXD") (pinfunction "Pin_2") (pintype "passive"))
+    (pad "3" thru_hole oval (at 0 5.08) (size 1.7 1.7) (drill 1) (layers *.Cu *.Mask)
+      (net 4 "/RXD") (pinfunction "Pin_3") (pintype "passive"))
+    (pad "4" thru_hole oval (at 0 7.62) (size 1.7 1.7) (drill 1) (layers *.Cu *.Mask)
+      (net 8 "3V3") (pinfunction "Pin_4") (pintype "passive"))
+    (pad "5" thru_hole oval (at 0 10.16) (size 1.7 1.7) (drill 1) (layers *.Cu *.Mask)
+      (net 3 "/EN") (pinfunction "Pin_5") (pintype "passive"))
+    (pad "6" thru_hole oval (at 0 12.7) (size 1.7 1.7) (drill 1) (layers *.Cu *.Mask)
+      (net 2 "/GPIO0") (pinfunction "Pin_6") (pintype "passive"))
     (model "${KICAD6_3DMODEL_DIR}/Connector_PinHeader_2.54mm.3dshapes/PinHeader_1x06_P2.54mm_Vertical.wrl"
       (offset (xyz 0 0 0))
@@
       (net 11 "/Power Section/Vrec") (pinfunction "K") (pintype "passive"))
     (pad "2" smd rect (at 2 0 90) (size 2.5 1.8) (layers "F.Cu" "F.Paste" "F.Mask")
-      (net 42 "Net-(J4-Pad2)") (pinfunction "A") (pintype "passive"))
+      (net 42 "Net-(D1-Pad1)") (pinfunction "A") (pintype "passive"))
     (model "${KICAD6_3DMODEL_DIR}/Diode_SMD.3dshapes/D_SMA.wrl"
       (offset (xyz 0 0 0))
@@
       (net 44 "PROBE_BUS") (pinfunction "IO27") (pintype "bidirectional"))
     (pad "13" smd rect (at -8.5 6.985) (size 2 0.9) (layers "F.Cu" "F.Paste" "F.Mask")
-      (net 22 "unconnected-(U1-Pad13)") (pinfunction "IO14") (pintype "bidirectional"))
+      (net 22 "unconnected-(U1-Pad13)") (pinfunction "IO14") (pintype "bidirectional+no_connect"))
     (pad "14" smd rect (at -8.5 8.255) (size 2 0.9) (layers "F.Cu" "F.Paste" "F.Mask")
       (net 23 "unconnected-(U1-Pad14)") (pinfunction "IO12") (pintype "bidirectional+no_connect"))
@@
       (net 1 "GND") (pinfunction "GND") (pintype "passive"))
     (pad "16" smd rect (at -4.445 9.255 90) (size 2 0.9) (layers "F.Cu" "F.Paste" "F.Mask")
-      (net 24 "unconnected-(U1-Pad16)") (pinfunction "IO13") (pintype "bidirectional"))
+      (net 24 "unconnected-(U1-Pad16)") (pinfunction "IO13") (pintype "bidirectional+no_connect"))
     (pad "17" smd rect (at -3.175 9.255 90) (size 2 0.9) (layers "F.Cu" "F.Paste" "F.Mask")
       (net 25 "unconnected-(U1-Pad17)") (pinfunction "SHD/SD2") (pintype "bidirectional+no_connect"))
@@
       (net 33 "unconnected-(U1-Pad26)") (pinfunction "IO4") (pintype "bidirectional+no_connect"))
     (pad "27" smd rect (at 8.5 5.715) (size 2 0.9) (layers "F.Cu" "F.Paste" "F.Mask")
-      (net 34 "unconnected-(U1-Pad27)") (pinfunction "IO16") (pintype "bidirectional"))
+      (net 34 "unconnected-(U1-Pad27)") (pinfunction "IO16") (pintype "bidirectional+no_connect"))
     (pad "28" smd rect (at 8.5 4.445) (size 2 0.9) (layers "F.Cu" "F.Paste" "F.Mask")
-      (net 35 "unconnected-(U1-Pad28)") (pinfunction "IO17") (pintype "bidirectional"))
+      (net 35 "unconnected-(U1-Pad28)") (pinfunction "IO17") (pintype "bidirectional+no_connect"))
     (pad "29" smd rect (at 8.5 3.175) (size 2 0.9) (layers "F.Cu" "F.Paste" "F.Mask")
       (net 36 "unconnected-(U1-Pad29)") (pinfunction "IO5") (pintype "bidirectional+no_connect"))
     (pad "30" smd rect (at 8.5 1.905) (size 2 0.9) (layers "F.Cu" "F.Paste" "F.Mask")
-      (net 54 "unconnected-(U1-Pad30)") (pinfunction "IO18") (pintype "bidirectional"))
+      (net 54 "unconnected-(U1-Pad30)") (pinfunction "IO18") (pintype "bidirectional+no_connect"))
     (pad "31" smd rect (at 8.5 0.635) (size 2 0.9) (layers "F.Cu" "F.Paste" "F.Mask")
-      (net 37 "unconnected-(U1-Pad31)") (pinfunction "IO19") (pintype "bidirectional"))
+      (net 37 "unconnected-(U1-Pad31)") (pinfunction "IO19") (pintype "bidirectional+no_connect"))
     (pad "32" smd rect (at 8.5 -0.635) (size 2 0.9) (layers "F.Cu" "F.Paste" "F.Mask")
       (net 38 "unconnected-(U1-Pad32)") (pinfunction "NC") (pintype "no_connect"))
     (pad "33" smd rect (at 8.5 -1.905) (size 2 0.9) (layers "F.Cu" "F.Paste" "F.Mask")
-      (net 39 "unconnected-(U1-Pad33)") (pinfunction "IO21") (pintype "bidirectional"))
+      (net 39 "unconnected-(U1-Pad33)") (pinfunction "IO21") (pintype "bidirectional+no_connect"))
     (pad "34" smd rect (at 8.5 -3.175) (size 2 0.9) (layers "F.Cu" "F.Paste" "F.Mask")
       (net 4 "/RXD") (pinfunction "RXD0/IO3") (pintype "bidirectional"))
@@
       (net 5 "/TXD") (pinfunction "TXD0/IO1") (pintype "bidirectional"))
     (pad "36" smd rect (at 8.5 -5.715) (size 2 0.9) (layers "F.Cu" "F.Paste" "F.Mask")
-      (net 40 "unconnected-(U1-Pad36)") (pinfunction "IO22") (pintype "bidirectional"))
+      (net 40 "unconnected-(U1-Pad36)") (pinfunction "IO22") (pintype "bidirectional+no_connect"))
     (pad "37" smd rect (at 8.5 -6.985) (size 2 0.9) (layers "F.Cu" "F.Paste" "F.Mask")
       (net 41 "unconnected-(U1-Pad37)") (pinfunction "IO23") (pintype "bidirectional+no_connect"))
@@
     (fp_line (start 2.3 -1.5) (end -2.3 -1.5) (layer "F.Fab") (width 0.1))
     (pad "1" smd rect (at -2 0) (size 2.5 1.8) (layers "F.Cu" "F.Paste" "F.Mask")
-      (net 42 "Net-(J4-Pad2)") (pinfunction "K") (pintype "passive"))
+      (net 42 "Net-(D1-Pad1)") (pinfunction "K") (pintype "passive"))
     (pad "2" smd rect (at 2 0) (size 2.5 1.8) (layers "F.Cu" "F.Paste" "F.Mask")
       (net 1 "GND") (pinfunction "A") (pintype "passive"))

Commit message: silkscreen for eflashy32
Other:
- board text added: "GND TXD RXD 3V3 EN GP0"
Changed lines of the file:
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@@
     (effects (font (size 0.8128 0.8128) (thickness 0.1524)) (justify mirror))
+  )
+  (gr_text "GND\n\nTXD\n\nRXD\n\n3V3\n\nEN\n\nGP0" (at 124.1 52.9) (layer "B.SilkS")
+    (effects (font (size 0.79 0.79) (thickness 0.1)) (justify right mirror))
   )
   (gr_text "+ T - + T - + T - + T -" (at 56.1 75.4) (layer "F.SilkS")
@@
     (effects (font (size 1.524 1.524) (thickness 0.3048)))
   )
+  (gr_text "GND\n\nTXD\n\nRXD\n\n3V3\n\nEN\n\nGP0" (at 118.7 52.9) (layer "F.SilkS")
+    (effects (font (size 0.79 0.79) (thickness 0.1)) (justify right))
+  )
   (gr_text "+ T - + T - + T - + T -" (at 87.9 75.4) (layer "F.SilkS")
