File: pcb/esptemp8c.kicad_pcb (KiCad board)
At the start: 2 copper layers, 98 x 50 mm, 39 parts, among them J1 Probes, J2 Probes, J3 eflashy32, J4 24VAC, J5 USB_C_Receptacle_USB2.0, U1 ESP32-WROOM-32D, U2 BD9G101G, U3 AMS1117-3.3

Commit message: updates for v2
Parts:
- removed C13: 1uF, Capacitor_SMD:C_0603_1608Metric
- removed FB1: 600@100MHz, Inductor_SMD:L_0805_2012Metric
- removed J4: 24VAC, Connector_Phoenix_MSTB:PhoenixContact_MSTBA_2,5_2-G-5,08_1x02_P5.08mm_Horizontal
- removed U3: AMS1117-3.3, Package_TO_SOT_SMD:SOT-223-3_TabPin2
- added D6: SS210, Diode_SMD:D_SMA, F.Cu at (50.5, 62.5)
- added D7: PWR, LED_SMD:LED_0805_2012Metric, F.Cu at (72.9, 61.1)
- added R7: 68k, Resistor_SMD:R_0402_1005Metric, F.Cu at (57.0, 59.5)
- added R8: 22k, Resistor_SMD:R_0402_1005Metric, F.Cu at (56.0, 59.5)
- added R9: 680, Resistor_SMD:R_0402_1005Metric, F.Cu at (73.9, 58.6)
- added SW1: RESET, Button_Switch_SMD:SW_Push_1P1T_XKB_TS-1187A, F.Cu at (104.0, 61.5)
- C1: value 10uF -> 10u
- C10: value 0.1uF 50V -> 0.1u
- C11, C12, C7: value 10uF 50V -> 10u; footprint Capacitor_SMD:C_1206_3216Metric -> Capacitor_SMD:C_0805_2012Metric
- C2: value 15nF -> 0.1u
- C8: value 47u -> 4u7
- C9: value 47u -> 0.1u; footprint Capacitor_SMD:C_1206_3216Metric -> Capacitor_SMD:C_0603_1608Metric
- D5: value SS210 -> CUS05S40.H3F; footprint Diode_SMD:D_SMA -> Diode_SMD:D_SOD-323
- J3: value eflashy32 -> 24VAC; footprint Connector_PinHeader_2.54mm:PinHeader_1x06_P2.54mm_Vertical -> Connector_Phoenix_MC:PhoenixContact_MC_1,5_2-G-3.81_1x02_P3.81mm_Horizontal
- L1: value 6.8uH -> 15uH; footprint Inductor_SMD:L_Sunlord_SWPA60xxS -> Inductor_SMD:L_Sunlord_SWPA6028S
- R3: value 3k9 -> 10k
- R4: value 680 -> 10k
- U1: value ESP32-WROOM-32D -> ESP32-C3-MINI-1; footprint RF_Module:ESP32-WROOM-32 -> Espressif:ESP32-C3-MINI-1
- U2: value BD9G101G -> LMR54406DBVR; footprint Package_TO_SOT_SMD:SOT-23-6 -> Package_TO_SOT_SMD:TSOT-23-6
- moved J3 56.2 mm to (65.3, 39.0), turned to 180 degrees
- moved R4 52.2 mm to (106.8, 53.4), turned to 90 degrees
- moved C7 42.3 mm to (93.0, 44.5), turned to 90 degrees
- moved R3 40.1 mm to (94.5, 51.0), turned to 0 degrees
- moved C2 36.9 mm to (95.0, 44.0), turned to 90 degrees
- moved D5 21.2 mm to (73.9, 48.4), turned to 90 degrees
- moved C8 15.4 mm to (53.7, 66.0), turned to -90 degrees
- moved R2 13.1 mm to (104.5, 53.5)
- moved C9 12.8 mm to (56.0, 65.2), turned to 90 degrees
- moved C1 7.48 mm to (88.5, 49.5), turned to 0 degrees
- moved U1 7.29 mm to (103.8, 42.7)
- moved C10 6.59 mm to (61.7, 63.1), turned to 90 degrees
- moved C11 3.57 mm to (74.3, 67.1), turned to -90 degrees
- moved C12 3.37 mm to (71.8, 67.1), turned to -90 degrees
- moved R1 3.16 mm to (89.0, 47.5), turned to 0 degrees
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Connections:
- net /Power Section/Vrec renamed Net-(D2-K)
- C1 pad 2: 3V3 -> /EN
- C10 pad 1: +5V -> /Power Section/LX
- C10 pad 2: /Power Section/FB -> /Power Section/BST
- C2 pad 1: Net-(C2-Pad1) -> GND
- C2 pad 2: /Power Section/LX -> 3V3
- C7 pad 1: Net-(C7-Pad1) -> GND
- C7 pad 2: GND -> 3V3
- C8 pad 1: +5V -> /Power Section/VIN
- C9 pad 1: +5V -> GND
- C9 pad 2: GND -> /Power Section/VIN
- D1 pad 1: Net-(D1-Pad1) -> Net-(D1-K)
- D2 pad 2: Net-(D1-Pad1) -> Net-(D1-K)
- D5 pad 1: /Power Section/LX -> /Power Section/VIN
- D5 pad 2: GND -> /Power Section/VBUS
- F1 pad 1: Net-(F1-Pad1) -> Net-(J3-Pin_1)
- J3 pad 1: GND -> Net-(J3-Pin_1)
- J3 pad 2: /TXD -> Net-(D1-K)
- J5 pad A4: +5V -> /Power Section/VBUS
- J5 pad A6: unconnected-(J5-PadA6) -> D+
- J5 pad A7: unconnected-(J5-PadA7) -> D-
- J5 pad A9: +5V -> /Power Section/VBUS
- J5 pad B4: +5V -> /Power Section/VBUS
- J5 pad B6: unconnected-(J5-PadB6) -> D+
- J5 pad B7: unconnected-(J5-PadB7) -> D-
- J5 pad B9: +5V -> /Power Section/VBUS
- L1 pad 2: +5V -> 3V3
- R1 pad 1: /EN -> 3V3
- R1 pad 2: 3V3 -> /EN
- R3 pad 1: /Power Section/FB -> 3V3
- R3 pad 2: +5V -> Net-(U1-GPIO2/ADC1_CH2)
- R4 pad 1: GND -> 3V3
- R4 pad 2: /Power Section/FB -> Net-(U1-GPIO8)
- U1 pad 11: unconnected-(U1-Pad11) -> GND
- U1 pad 12: PROBE_BUS -> unconnected-(U1-GPIO0/ADC1_CH0/XTAL_32K_P-Pad12)
- U1 pad 14: unconnected-(U1-Pad14) -> GND
- U1 pad 15: GND -> unconnected-(U1-NC-Pad15)
- U1 pad 2: 3V3 -> GND
- U1 pad 20: unconnected-(U1-Pad20) -> PROBE_BUS
- U1 pad 22: unconnected-(U1-Pad22) -> Net-(U1-GPIO8)
- U1 pad 23: unconnected-(U1-Pad23) -> /GPIO0
- U1 pad 25: /GPIO0 -> unconnected-(U1-NC-Pad25)
- U1 pad 26: unconnected-(U1-Pad26) -> D-
- U1 pad 27: unconnected-(U1-Pad27) -> D+
- U1 pad 3: /EN -> 3V3
- U1 pad 34: /RXD -> unconnected-(U1-NC-Pad34)
- U1 pad 35: /TXD -> unconnected-(U1-NC-Pad35)
- U1 pad 36: unconnected-(U1-Pad36) -> GND
- U1 pad 37: unconnected-(U1-Pad37) -> GND
- U1 pad 5: unconnected-(U1-Pad5) -> Net-(U1-GPIO2/ADC1_CH2)
- U1 pad 8: unconnected-(U1-Pad8) -> /EN
- U2 pad 1: Net-(C2-Pad1) -> /Power Section/BST
- U2 pad 3: /Power Section/FB -> /Power Section/FB2
- U2 pad 4: Net-(C7-Pad1) -> /Power Section/VIN
- U2 pad 5: Net-(C7-Pad1) -> /Power Section/VIN
Routing:
- net +5V: track 107.2 -> 0.00 mm, vias 5 -> 0
- net D+: track 0.00 -> 66.6 mm
- net D-: track 0.00 -> 61.6 mm, vias 0 -> 2
- net GND: track 101.5 -> 41.4 mm, vias 28 -> 24
- net /Power Section/VIN: track 0.00 -> 58.9 mm
- net /EN: track 49.5 -> 10.7 mm, vias 1 -> 0
- net Net-(C7-Pad1): track 35.1 -> 0.00 mm
- net 3V3: track 180.9 -> 203.7 mm, vias 5 -> 4
- net /Power Section/VBUS: track 0.00 -> 19.1 mm
- net Net-(D1-K): track 0.00 -> 18.5 mm
- net Net-(D1-Pad1): track 12.6 -> 0.00 mm
- net PROBE_BUS: track 97.1 -> 107.8 mm, vias 0 -> 2
- net /RXD: track 10.5 -> 0.00 mm
- net /TXD: track 9.73 -> 0.00 mm
- net Net-(J3-Pin_1): track 0.00 -> 9.17 mm
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Other:
- board text added: "<<hash>>"
- board text added: "esptemp8c v2"
- board text removed: "Do not connect both power inputs"
- board text removed: "GND TXD RXD 3V3 EN GP0"
- board text removed: "eflashy32"
- board text removed: "esptemp8c"

Commit message: more v2 changes
Parts:
- removed D6: SS210, Diode_SMD:D_SMA
- added J4: T3, Connector_Phoenix_MC:PhoenixContact_MC_1,5_3-G-3.81_1x03_P3.81mm_Horizontal, F.Cu at (71.5, 152.6)
- added J6: T4, Connector_Phoenix_MC:PhoenixContact_MC_1,5_3-G-3.81_1x03_P3.81mm_Horizontal, F.Cu at (85.5, 152.6)
- D1, D2, D3, D4: value SS210 -> 1N5819WS; footprint Diode_SMD:D_SMA -> Diode_SMD:D_SOD-323
- J1: value Probes -> T1; footprint TerminalBlock_Phoenix:TerminalBlock_Phoenix_MPT-0,5-12-2.54_1x12_P2.54mm_Horizontal -> Connector_Phoenix_MC:PhoenixContact_MC_1,5_3-G-3.81_1x03_P3.81mm_Horizontal
- J2: value Probes -> T2; footprint TerminalBlock_Phoenix:TerminalBlock_Phoenix_MPT-0,5-12-2.54_1x12_P2.54mm_Horizontal -> Connector_Phoenix_MC:PhoenixContact_MC_1,5_3-G-3.81_1x03_P3.81mm_Horizontal
- moved H4 86.1 mm to (82.3, 114.8)
- moved R4 83.0 mm to (59.8, 121.8), turned to 0 degrees
- moved R2 80.6 mm to (59.8, 120.5)
- moved J2 78.4 mm to (57.5, 152.6)
- moved R3 76.6 mm to (59.7, 119.2)
- moved H3 76.2 mm to (54.3, 114.8)
- moved C4 75.8 mm to (50.5, 126.2), turned to -90 degrees
- moved H2 75.2 mm to (82.3, 142.8)
- moved U1 74.9 mm to (68.4, 108.7)
- moved C5 73.6 mm to (53.0, 121.5), turned to 90 degrees
- moved D5 73.5 mm to (90.7, 120.0)
- moved C3 73.1 mm to (53.0, 126.2), turned to -90 degrees
- moved J1 73.0 mm to (43.5, 152.6)
- moved C2 72.9 mm to (60.0, 108.0), turned to -90 degrees
- moved D3 72.9 mm to (46.4, 124.0), turned to 0 degrees
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Connections:
- net /GPIO0 renamed /GPIO9
- C3 pad 1: Net-(D2-K) -> /Power Section/VIN
- C4 pad 1: Net-(D2-K) -> /Power Section/VIN
- C5 pad 1: Net-(D2-K) -> /Power Section/VIN
- C6 pad 1: Net-(D2-K) -> /Power Section/VIN
- D2 pad 1: Net-(D2-K) -> /Power Section/VIN
- D4 pad 1: Net-(D2-K) -> /Power Section/VIN
- F1 pad 1: Net-(J3-Pin_1) -> Net-(J3-Pin_2)
- F1 pad 2: Net-(D3-K) -> Net-(D1-K)
- J3 pad 1: Net-(J3-Pin_1) -> Net-(D3-K)
- J3 pad 2: Net-(D1-K) -> Net-(J3-Pin_2)
Routing:
- net 3V3: track 203.7 -> 138.0 mm, vias 4 -> 0
- net GND: track 41.4 -> 92.6 mm, vias 24 -> 32
- net /Power Section/VIN: track 58.9 -> 99.2 mm, vias 0 -> 2
- net D+: track 66.6 -> 27.0 mm
- net D-: track 61.6 -> 24.5 mm
- net Net-(D3-K): track 6.83 -> 33.4 mm
- net Net-(D2-K): track 26.3 -> 0.00 mm
- net Net-(D1-K): track 18.5 -> 4.54 mm
- net Net-(U1-GPIO8): track 2.65 -> 14.2 mm
- net Net-(J3-Pin_1): track 9.17 -> 0.00 mm
- net /EN: track 10.7 -> 4.00 mm
- net Net-(J3-Pin_2): track 0.00 -> 6.29 mm
- net PROBE_BUS: track 107.8 -> 101.9 mm, vias 2 -> 3
- net /Power Section/VBUS: track 19.1 -> 22.8 mm
- net /GPIO9: track 15.3 -> 11.9 mm, vias 2 -> 0
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Other:
- board size 98 x 50 mm -> 56.6 x 57.7 mm
- board text added: "140mA hold / 340mA trip mSMD014"
- board text added: "Case : Hammond 1593KBK"
- board text removed: "Case : Hammond 1593VBK"

Commit message: fix
Other:
- board text added: "JLCJLCJLCJLC1"
- board text removed: "JLCJLCJLCJLC"
Changed lines of the file:
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@@
 		)
 	)
-	(gr_text "JLCJLCJLCJLC"
+	(gr_text "JLCJLCJLCJLC1"
 		(at 88.744374 101 0)
 		(layer "F.SilkS")
