File: pcb/esptemp8c.kicad_pcb (KiCad board)
At the start: 2 copper layers, 56.6 x 57.7 mm, 42 parts, among them J1 T1, J2 T2, J3 24VAC, J4 T3, J5 USB_C_Receptacle_USB2.0, J6 T4, SW1 RESET, U1 ESP32-C3-MINI-1, U2 LMR54406DBVR

Commit message: docs and pics
Parts:
- D5: value CUS05S40.H3F -> 1N5819WS
Other:
- board text added: "3V SIG GND"
- board text removed: "+ T - + T - + T - + T -"
Changed lines of the file:
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@@
 			)
 		)
-		(property "Value" "CUS05S40.H3F"
+		(property "Value" "1N5819WS"
 			(at 0.1 1.9 90)
 			(layer "F.Fab")
@@
 			)
 		)
-		(property "LCSC" "C2762696"
+		(property "LCSC" "C191023"
 			(at -3.8 128.8 0)
 			(layer "F.Fab")
@@
 		)
 	)
-	(gr_text "+ T - + T - + T - + T -"
-		(at 43.994374 148.5 0)
-		(layer "F.SilkS")
+	(gr_text "<<hash>>"
+		(at 93.994374 132 -90)
+		(layer "B.SilkS")
+		(effects
+			(font
+				(size 1.524 1.524)
+				(thickness 0.3048)
+			)
+			(justify left bottom mirror)
+		)
+	)
+	(gr_text "3V\nSIG\nGND"
+		(at 56.494374 150.5 90)
+		(layer "F.SilkS" knockout)
+		(effects
+			(font
+				(size 2.2 2)
+				(thickness 0.3048)
+			)
+			(justify left top)
+		)
+	)
+	(gr_text "3V\nSIG\nGND"
+		(at 70.494374 150.5 90)
+		(layer "F.SilkS" knockout)
 		(effects
 			(font
-				(size 1.385 1.385)
+				(size 2.2 2)
 				(thickness 0.3048)
 			)
-			(justify left)
+			(justify left top)
+		)
+	)
+	(gr_text "3V\nSIG\nGND"
+		(at 42.494374 150.5 90)
+		(layer "F.SilkS" knockout)
+		(effects
+			(font
+				(size 2.2 2)
+				(thickness 0.3048)
+			)
+			(justify left top)
 		)
 	)
@@
 		)
 	)
+	(gr_text "3V\nSIG\nGND"
+		(at 84.494374 150.5 90)
+		(layer "F.SilkS" knockout)
+		(effects
+			(font
+				(size 2.2 2)
+				(thickness 0.3048)
+			)
+			(justify left top)
+		)
+	)
 	(gr_text "JLCJLCJLCJLC1"
 		(at 88.744374 101 0)
@@
 		)
 	)
-	(gr_text "<<hash>>"
-		(at 95.744374 132.5 90)
-		(layer "F.SilkS")
-		(effects
-			(font
-				(size 1.524 1.524)
-				(thickness 0.3048)
-			)
-			(justify left bottom)
-		)
-	)

Commit message: final touches and check
Parts:
- U2: footprint Package_TO_SOT_SMD:TSOT-23-6 -> Package_TO_SOT_SMD:SOT-23-6
Changed lines of the file:
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@@
 		)
 	)
-	(footprint "Package_TO_SOT_SMD:TSOT-23-6"
+	(footprint "Package_TO_SOT_SMD:SOT-23-6"
 		(layer "F.Cu")
 		(at 54.494374 133.5 -90)
-		(descr "TSOT, 6 Pin (https://www.jedec.org/sites/default/files/docs/MO-193D.pdf variant AA), generated with kicad-footprint-generator ipc_gullwing_generator.py")
-		(tags "TSOT TO_SOT_SMD")
+		(descr "SOT, 6 Pin (https://www.jedec.org/sites/default/files/docs/Mo-178c.PDF variant AB), generated with kicad-footprint-generator ipc_gullwing_generator.py")
+		(tags "SOT TO_SOT_SMD")
 		(property "Reference" "U2"
-			(at 0 -2.4 -90)
+			(at 0 -2.4 270)
 			(layer "F.SilkS")
 			(hide yes)
@@
 			)
 		)
-		(property "Footprint" "Package_TO_SOT_SMD:TSOT-23-6"
+		(property "Footprint" "Package_TO_SOT_SMD:SOT-23-6"
 			(at 0 0 -90)
+			(unlocked yes)
 			(layer "F.Fab")
 			(hide yes)
@@
 		(property "Datasheet" "http://www.ti.com/lit/ds/symlink/lm2842-q1.pdf"
 			(at 0 0 -90)
+			(unlocked yes)
 			(layer "F.Fab")
 			(hide yes)
@@
 		(property "Description" ""
 			(at 0 0 -90)
+			(unlocked yes)
 			(layer "F.Fab")
 			(hide yes)
@@
 			)
 		)
+		(property "Notes" ""
+			(at 0 0 -90)
+			(unlocked yes)
+			(layer "F.Fab")
+			(hide yes)
+			(effects
+				(font
+					(size 1 1)
+					(thickness 0.15)
+				)
+			)
+		)
 		(property ki_fp_filters "TSOT?23*")
 		(sheetname "Power Section")
@@
 			(pintype "output")
 		)
-		(model "${KICAD8_3DMODEL_DIR}/Package_TO_SOT_SMD.3dshapes/TSOT-23-6.wrl"
+		(model "${KICAD8_3DMODEL_DIR}/Package_TO_SOT_SMD.3dshapes/SOT-23-6.wrl"
 			(offset
 				(xyz 0 0 0)
@@
 	)
 	(gr_text "<<hash>>"
-		(at 93.994374 132 -90)
+		(at 93.994374 132 270)
 		(layer "B.SilkS")
 		(effects
 			(font
-				(size 1.524 1.524)
-				(thickness 0.3048)
+				(size 1.2 1.2)
+				(thickness 0.2)
+				(bold yes)
 			)
 			(justify left bottom mirror)
@@
 	)
 	(gr_text "esptemp8c\nv2"
-		(at 73.494374 134.25 0)
+		(at 75.494374 132.5 0)
 		(layer "F.SilkS")
 		(effects
@@
 	)
 	(segment
-		(start 87.572454 111.4385)
-		(end 84.666294 111.4385)
+		(start 76.872454 114.3885)
+		(end 75.105875 114.3885)
 		(width 0.127)
 		(layer "F.Cu")
@@
 	)
 	(segment
-		(start 88.3685 108.744001)
-		(end 88.3685 110.642454)
+		(start 84.666294 111.4385)
+		(end 83.416294 110.1885)
 		(width 0.127)
 		(layer "F.Cu")
@@
 	)
 	(segment
-		(start 81.072454 110.1885)
-		(end 76.822454 114.4385)
-		(width 0.127)
-		(layer "F.Cu")
-		(net 33)
-	)
-	(segment
 		(start 89.43 105.997027)
 		(end 89.43 107.595)
@@
 	)
 	(segment
-		(start 75.600104 114.4385)
-		(end 75.550104 114.3885)
+		(start 75.105875 114.3885)
+		(end 74.894375 114.6)
 		(width 0.127)
 		(layer "F.Cu")
@@
 	)
 	(segment
-		(start 83.416294 110.1885)
-		(end 81.072454 110.1885)
+		(start 88.3685 108.744001)
+		(end 88.3685 110.642454)
 		(width 0.127)
 		(layer "F.Cu")
@@
 	)
 	(segment
-		(start 88.43 107.595)
-		(end 88.43 108.682501)
-		(width 0.127)
-		(layer "F.Cu")
-		(net 33)
-	)
-	(segment
-		(start 75.550104 114.3885)
-		(end 75.105875 114.3885)
+		(start 83.416294 110.1885)
+		(end 81.072454 110.1885)
 		(width 0.127)
 		(layer "F.Cu")
@@
 	)
 	(segment
-		(start 88.43 108.682501)
-		(end 88.3685 108.744001)
+		(start 88.3685 110.642454)
+		(end 87.572454 111.4385)
 		(width 0.127)
 		(layer "F.Cu")
@@
 	)
 	(segment
-		(start 76.822454 114.4385)
-		(end 75.600104 114.4385)
+		(start 88.43 107.595)
+		(end 88.43 108.682501)
 		(width 0.127)
 		(layer "F.Cu")
@@
 	)
 	(segment
-		(start 88.3685 110.642454)
-		(end 87.572454 111.4385)
+		(start 88.43 108.682501)
+		(end 88.3685 108.744001)
 		(width 0.127)
 		(layer "F.Cu")
@@
 	)
 	(segment
-		(start 84.666294 111.4385)
-		(end 83.416294 110.1885)
+		(start 87.572454 111.4385)
+		(end 84.666294 111.4385)
 		(width 0.127)
 		(layer "F.Cu")
@@
 	)
 	(segment
-		(start 75.105875 114.3885)
-		(end 74.894375 114.6)
+		(start 81.072454 110.1885)
+		(end 76.872454 114.3885)
 		(width 0.127)
 		(layer "F.Cu")
@@
 	)
 	(segment
+		(start 83.572454 109.8115)
+		(end 80.916294 109.8115)
+		(width 0.127)
+		(layer "F.Cu")
+		(net 34)
+	)
+	(segment
 		(start 88.758824 104.174413)
 		(end 88.139524 104.174413)
@@
 	)
 	(segment
-		(start 87.93 108.682501)
-		(end 87.9915 108.744001)
-		(width 0.127)
-		(layer "F.Cu")
-		(net 34)
-	)
-	(segment
-		(start 80.916294 109.8115)
-		(end 76.666294 114.0615)
-		(width 0.127)
-		(layer "F.Cu")
-		(net 34)
-	)
-	(segment
-		(start 84.822454 111.0615)
-		(end 83.572454 109.8115)
-		(width 0.127)
-		(layer "F.Cu")
-		(net 34)
-	)
-	(segment
-		(start 75.744374 114.0615)
-		(end 75.694374 114.0115)
+		(start 87.9915 108.744001)
+		(end 87.9915 110.486294)
 		(width 0.127)
 		(layer "F.Cu")
@@
 	)
 	(segment
-		(start 74.894375 113.8)
-		(end 74.294374 113.8)
+		(start 76.716294 114.0115)
+		(end 75.105875 114.0115)
 		(width 0.127)
 		(layer "F.Cu")
@@
 	)
 	(segment
-		(start 76.666294 114.0615)
-		(end 75.744374 114.0615)
+		(start 87.93 108.682501)
+		(end 87.9915 108.744001)
 		(width 0.127)
 		(layer "F.Cu")
@@
 	)
 	(segment
-		(start 87.9915 108.744001)
-		(end 87.9915 110.486294)
+		(start 87.866065 107.531065)
+		(end 87.93 107.595)
 		(width 0.127)
 		(layer "F.Cu")
@@
 	)
 	(segment
-		(start 75.694374 114.0115)
-		(end 75.105875 114.0115)
+		(start 89.000609 106.63013)
+		(end 89.000609 104.416198)
 		(width 0.127)
 		(layer "F.Cu")
@@
 	)
 	(segment
-		(start 87.866065 107.531065)
-		(end 87.93 107.595)
+		(start 87.416294 111.0615)
+		(end 84.822454 111.0615)
 		(width 0.127)
 		(layer "F.Cu")
@@
 	)
 	(segment
-		(start 89.000609 106.63013)
-		(end 89.000609 104.416198)
+		(start 89.000609 104.416198)
+		(end 88.758824 104.174413)
 		(width 0.127)
 		(layer "F.Cu")
@@
 	)
 	(segment
-		(start 89.000609 104.416198)
-		(end 88.758824 104.174413)
+		(start 80.916294 109.8115)
+		(end 76.716294 114.0115)
 		(width 0.127)
 		(layer "F.Cu")
@@
 	)
 	(segment
-		(start 83.572454 109.8115)
-		(end 80.916294 109.8115)
+		(start 74.894375 113.8)
+		(end 74.294374 113.8)
 		(width 0.127)
 		(layer "F.Cu")
@@
 	)
 	(segment
-		(start 75.105875 114.0115)
-		(end 74.894375 113.8)
+		(start 88.139524 104.174413)
+		(end 87.866065 104.447872)
 		(width 0.127)
 		(layer "F.Cu")
@@
 	)
 	(segment
-		(start 87.416294 111.0615)
-		(end 84.822454 111.0615)
+		(start 84.822454 111.0615)
+		(end 83.572454 109.8115)
 		(width 0.127)
 		(layer "F.Cu")
@@
 	)
 	(segment
-		(start 88.139524 104.174413)
-		(end 87.866065 104.447872)
+		(start 75.105875 114.0115)
+		(end 74.894375 113.8)
 		(width 0.127)
 		(layer "F.Cu")
