File: pcb/esptemp8c-power.kicad_sch (KiCad schematic)
At the start: 27 parts, among them J4 24VAC, J5 USB_C_Receptacle_USB2.0, U2 BD9G101G, U3 AMS1117-3.3

Commit message: updates for v2
Parts:
- removed C2: 15nF, Capacitor_SMD:C_0603_1608Metric, symbol Device:C_Small
- removed C7: 10uF 50V, Capacitor_SMD:C_1206_3216Metric, symbol Device:C_Small
- removed FB1: 600@100MHz, Inductor_SMD:L_0805_2012Metric, symbol Device:FerriteBead_Small
- removed J4: 24VAC, Connector_Phoenix_MSTB:PhoenixContact_MSTBA_2,5_2-G-5,08_1x02_P5.08mm_Horizontal, symbol Connector:Screw_Terminal_01x02
- removed R3: 3k9, Resistor_SMD:R_0402_1005Metric, symbol Device:R_Small
- removed R4: 680, Resistor_SMD:R_0402_1005Metric, symbol Device:R_Small
- removed U2: BD9G101G, Package_TO_SOT_SMD:SOT-23-6, symbol Regulator_Switching:AOZ1280CI
- removed U3: AMS1117-3.3, Package_TO_SOT_SMD:SOT-223-3_TabPin2, symbol Regulator_Linear:AP1117-33
- added D6: SS210, Diode_SMD:D_SMA, symbol Device:D_Schottky_Small
- added J3: 24VAC, Connector_Phoenix_MC:PhoenixContact_MC_1,5_2-G-3.81_1x02_P3.81mm_Horizontal, symbol Connector:Screw_Terminal_01x02
- added R7: 68k, Resistor_SMD:R_0402_1005Metric, symbol Device:R_Small
- added R8: 22k, Resistor_SMD:R_0402_1005Metric, symbol Device:R_Small
- added TP1, TP2: TP_VIN, Connector_PinHeader_2.54mm:PinHeader_1x01_P2.54mm_Vertical, symbol Connector:TestPoint
- added U2: LMR54406DBVR, Package_TO_SOT_SMD:TSOT-23-6, symbol Regulator_Switching:LM2840X
- C10: value 0.1uF 50V -> 0.1u
- C11, C12: value 10uF 50V -> 10u; footprint Capacitor_SMD:C_1206_3216Metric -> Capacitor_SMD:C_0805_2012Metric; LCSC C13585 -> C15850
- C8: value 47u -> 4u7; LCSC C96123 -> C29823
- C9: value 47u -> 0.1u; footprint Capacitor_SMD:C_1206_3216Metric -> Capacitor_SMD:C_0603_1608Metric; LCSC C96123 -> C14663
- D5: value SS210 -> CUS05S40.H3F; footprint Diode_SMD:D_SMA -> Diode_SMD:D_SOD-323; LCSC C14996 -> C2762696
- J5: symbol Connector:USB_C_Receptacle_USB2.0 -> Connector:USB_C_Receptacle_USB2.0_16P
- L1: value 6.8uH -> 15uH; footprint Inductor_SMD:L_Sunlord_SWPA60xxS -> Inductor_SMD:L_Sunlord_SWPA6028S; LCSC C57254 -> C83373; PN (none) -> SRN6045-150M or SWPA6045S150MT
Connections:
- net +3V3: now also L1.2, R7.2, TP2.1
- net GND: now also C9.1, R8.2, U2.2 (GND); no longer C9.2, D5.2 (A)
- net LX: now also C10.1, TP1.1, U2.6 (SW); no longer D5.1 (K)
- net D+: now reaches J5.A6 (D+)
- net D+: now also J5.B6 (D+)
- net D-: now reaches J5.A7 (D-)
- net D-: now also J5.B7 (D-)
- net at F1.1: now also J3.1 (Pin_1)
- net at D1.1 (K), D2.2 (A): now also J3.2 (Pin_2)
- net +5V renamed VBUS
- net VBUS: now also D5.2 (A); no longer C10.1, C8.1, C9.1, L1.2
- net FB renamed BST
- net BST: now also U2.1 (BOOST)
- net Vrec: no longer names the net of C3.1, C4.1, C5.1, C6.1, D2.1 (K), D4.1 (K)
- net Vrec: now also D6.2 (A)
- new net FB2: R7.1, R8.1, U2.3 (FB)
- new net VIN: C8.1, C9.2, D5.1 (K), D6.1 (K), U2.4 (EN), U2.5 (VIN)
- no-connect marks 7 -> 3
Other:
- note added: "24VAC->3V Regulation (500mA max)"
- note removed: "24VAC->5VDC Regulation (500mA max)"
- note removed: "5VDC Regulation"
- note removed: "Alternate 5VDC Source"
- moved on the sheet: C3, C4, C5, C6, D1, D2, D3, D4, F1, J5, R5, R6

Commit message: more v2 changes
Parts:
- removed D6: SS210, Diode_SMD:D_SMA, symbol Device:D_Schottky_Small
- D1, D2, D3, D4: value SS210 -> 1N5819WS; footprint Diode_SMD:D_SMA -> Diode_SMD:D_SOD-323; LCSC C14996 -> C191023
Connections:
- net VIN: now also C3.1, C4.1, C5.1, C6.1, D2.1 (K), D4.1 (K)
- net at D3.1 (K), D4.2 (A): now also J3.1 (Pin_1); no longer F1.2
- net at D1.1 (K), D2.2 (A): now also F1.2; no longer J3.2 (Pin_2)
- net at F1.1: now also J3.2 (Pin_2); no longer J3.1 (Pin_1)
Other:
- moved on the sheet: F1
Changed lines of the file:
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@@
 	(wire
 		(pts
-			(xy 133.35 73.66) (xy 135.89 73.66)
+			(xy 133.35 73.66) (xy 142.24 73.66)
 		)
 		(stroke
@@
 	(wire
 		(pts
+			(xy 87.63 72.39) (xy 92.71 72.39)
+		)
+		(stroke
+			(width 0)
+			(type default)
+		)
+	)
+	(wire
+		(pts
 			(xy 107.95 66.04) (xy 107.95 71.12)
 		)
@@
 	(wire
 		(pts
-			(xy 76.2 74.93) (xy 82.55 74.93)
+			(xy 76.2 74.93) (xy 92.71 74.93)
 		)
 		(stroke
@@
 	(wire
 		(pts
-			(xy 140.97 73.66) (xy 142.24 73.66)
-		)
-		(stroke
-			(width 0)
-			(type default)
-		)
-	)
-	(wire
-		(pts
 			(xy 107.95 81.28) (xy 92.71 81.28)
 		)
@@
 	(wire
 		(pts
-			(xy 87.63 74.93) (xy 92.71 74.93)
-		)
-		(stroke
-			(width 0)
-			(type default)
-		)
-	)
-	(wire
-		(pts
 			(xy 224.79 83.82) (xy 219.71 83.82)
 		)
@@
 	(wire
 		(pts
-			(xy 76.2 72.39) (xy 92.71 72.39)
+			(xy 76.2 72.39) (xy 82.55 72.39)
 		)
 		(stroke
@@
 	)
 	(symbol
-		(lib_id "Device:D_Schottky_Small")
-		(at 138.43 73.66 180)
-		(unit 1)
-		(exclude_from_sim no)
-		(in_bom yes)
-		(on_board yes)
-		(dnp no)
-		(fields_autoplaced yes)
-		(property "Reference" "D6"
-			(at 138.684 70.485 0)
-			(effects
-				(font
-					(size 1.27 1.27)
-				)
-			)
-		)
-		(property "Value" "SS210"
-			(at 138.684 69.85 0)
-			(effects
-				(font
-					(size 1.27 1.27)
-				)
-				(hide yes)
-			)
-		)
-		(property "Footprint" "Diode_SMD:D_SMA"
-			(at 138.43 73.66 90)
-			(effects
-				(font
-					(size 1.27 1.27)
-				)
-				(hide yes)
-			)
-		)
-		(property "Datasheet" "~"
-			(at 138.43 73.66 90)
-			(effects
-				(font
-					(size 1.27 1.27)
-				)
-				(hide yes)
-			)
-		)
-		(property "Description" ""
-			(at 138.43 73.66 0)
-			(effects
-				(font
-					(size 1.27 1.27)
-				)
-				(hide yes)
-			)
-		)
-		(property "LCSC" "C14996"
-			(at 138.43 73.66 0)
-			(effects
-				(font
-					(size 1.27 1.27)
-				)
-				(hide yes)
-			)
-		)
-		(pin "1"
-		)
-		(pin "2"
-		)
-		(instances
-			(project "esptemp8c"
-				(path "/23e49c1c-e106-44cc-bc49-1a732eea896b/9514ff5c-b9a3-4b17-b039-8821c46f7fb4"
-					(reference "D6")
-					(unit 1)
-				)
-			)
-		)
-	)
-	(symbol
 		(lib_id "Device:R_Small")
 		(at 120.65 109.22 0)
@@
 			)
 		)
-		(property "Value" "SS210"
+		(property "Value" "1N5819WS"
 			(at 104.394 73.66 0)
 			(effects
@@
 			)
 		)
-		(property "Footprint" "Diode_SMD:D_SMA"
+		(property "Footprint" "Diode_SMD:D_SOD-323"
 			(at 104.14 77.47 90)
 			(effects
@@
 			)
 		)
-		(property "LCSC" "C14996"
+		(property "LCSC" "C191023"
 			(at 104.14 77.47 0)
 			(effects
@@
 			)
 		)
-		(property "Value" "SS210"
+		(property "Value" "1N5819WS"
 			(at 112.014 67.31 0)
 			(effects
@@
 			)
 		)
-		(property "Footprint" "Diode_SMD:D_SMA"
+		(property "Footprint" "Diode_SMD:D_SOD-323"
 			(at 111.76 71.12 90)
 			(effects
@@
 			)
 		)
-		(property "LCSC" "C14996"
+		(property "LCSC" "C191023"
 			(at 111.76 71.12 0)
 			(effects
@@
 	(symbol
 		(lib_id "Device:Polyfuse_Small")
-		(at 85.09 74.93 90)
+		(at 85.09 72.39 90)
 		(unit 1)
 		(exclude_from_sim no)
@@
 		(dnp no)
 		(property "Reference" "F1"
-			(at 85.09 68.58 90)
+			(at 85.09 66.04 90)
 			(effects
 				(font
@@
 		)
 		(property "Value" "140mA hold / 340mA trip mSMD014"
-			(at 85.09 71.12 90)
+			(at 85.09 68.58 90)
 			(effects
 				(font
@@
 		)
 		(property "Footprint" "Fuse:Fuse_1812_4532Metric"
-			(at 90.17 73.66 0)
+			(at 90.17 71.12 0)
 			(effects
 				(font
@@
 		)
 		(property "Datasheet" "~"
-			(at 85.09 74.93 0)
+			(at 85.09 72.39 0)
 			(effects
 				(font
@@
 		)
 		(property "Description" ""
-			(at 85.09 74.93 0)
+			(at 85.09 72.39 0)
 			(effects
 				(font
@@
 		)
 		(property "LCSC" "C70106"
-			(at 85.09 74.93 0)
+			(at 85.09 72.39 0)
 			(effects
 				(font
@@
 			)
 		)
-		(property "Value" "SS210"
+		(property "Value" "1N5819WS"
 			(at 104.394 67.31 0)
 			(effects
@@
 			)
 		)
-		(property "Footprint" "Diode_SMD:D_SMA"
+		(property "Footprint" "Diode_SMD:D_SOD-323"
 			(at 104.14 71.12 90)
 			(effects
@@
 			)
 		)
-		(property "LCSC" "C14996"
+		(property "LCSC" "C191023"
 			(at 104.14 71.12 0)
 			(effects
@@
 			)
 		)
-		(property "Value" "SS210"
+		(property "Value" "1N5819WS"
 			(at 112.014 73.66 0)
 			(effects
@@
 			)
 		)
-		(property "Footprint" "Diode_SMD:D_SMA"
+		(property "Footprint" "Diode_SMD:D_SOD-323"
 			(at 111.76 77.47 90)
 			(effects
@@
 			)
 		)
-		(property "LCSC" "C14996"
+		(property "LCSC" "C191023"
 			(at 111.76 77.47 0)
 			(effects

Commit message: docs and pics
Parts:
- D5: value CUS05S40.H3F -> 1N5819WS; LCSC C2762696 -> C191023
Changed lines of the file:
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@@
 			)
 		)
-		(property "Value" "CUS05S40.H3F"
+		(property "Value" "1N5819WS"
 			(at 125.984 97.79 0)
 			(effects
@@
 			)
 		)
-		(property "LCSC" "C2762696"
+		(property "LCSC" "C191023"
 			(at 125.73 101.6 0)
 			(effects

Commit message: fix footprint to sot23
Parts:
- U2: footprint Package_TO_SOT_SMD:TSOT-23-6 -> Package_TO_SOT_SMD:SOT-23-6
Changed lines of the file:
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@@
 			)
 		)
-		(property "Footprint" "Package_TO_SOT_SMD:TSOT-23-6"
+		(property "Footprint" "Package_TO_SOT_SMD:SOT-23-6"
 			(at 174.625 82.55 0)
 			(effects
@@
 			)
 		)
+		(property "Notes" ""
+			(at 173.99 76.2 0)
+			(effects
+				(font
+					(size 1.27 1.27)
+				)
+			)
+		)

Commit message: final touches and check
Changed lines of the file:
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@@
+	)
+	(junction
+		(at 118.11 115.57)
+		(diameter 0)
+		(color 0 0 0 0)
 	)
 	(junction
@@
 	(junction
 		(at 219.71 83.82)
-		(diameter 0)
-		(color 0 0 0 0)
-	)
-	(junction
-		(at 118.11 114.3)
 		(diameter 0)
 		(color 0 0 0 0)
@@
 	(wire
 		(pts
-			(xy 118.11 114.3) (xy 118.11 116.84)
+			(xy 118.11 115.57) (xy 118.11 116.84)
 		)
 		(stroke
@@
 	(wire
 		(pts
-			(xy 120.65 114.3) (xy 120.65 111.76)
+			(xy 120.65 115.57) (xy 120.65 111.76)
 		)
 		(stroke
@@
 	(wire
 		(pts
-			(xy 114.3 114.3) (xy 118.11 114.3)
+			(xy 114.3 115.57) (xy 118.11 115.57)
 		)
 		(stroke
@@
 	(wire
 		(pts
+			(xy 118.11 115.57) (xy 120.65 115.57)
+		)
+		(stroke
+			(width 0)
+			(type default)
+		)
+	)
+	(wire
+		(pts
 			(xy 142.24 73.66) (xy 144.78 73.66)
 		)
@@
 	(wire
 		(pts
-			(xy 118.11 114.3) (xy 120.65 114.3)
-		)
-		(stroke
-			(width 0)
-			(type default)
-		)
-	)
-	(wire
-		(pts
 			(xy 215.9 83.82) (xy 219.71 83.82)
 		)
@@
 	(wire
 		(pts
+			(xy 114.3 115.57) (xy 114.3 114.3)
+		)
+		(stroke
+			(width 0)
+			(type default)
+		)
+	)
+	(wire
+		(pts
 			(xy 95.25 73.66) (xy 95.25 74.93)
 		)
@@
 			(width 0)
 			(type default)
+		)
+	)
+	(rectangle
+		(start 60.96 63.5)
+		(end 236.22 147.32)
+		(stroke
+			(width 0)
+			(type default)
+		)
+		(fill
+			(type none)
 		)
 	)
 	(text "24VAC->3V Regulation (500mA max)"
 		(exclude_from_sim no)
-		(at 67.31 60.96 0)
+		(at 60.96 63.5 0)
 		(effects
 			(font
