File: pcb/esptemp8c.kicad_sch (KiCad schematic)
At the start: 12 parts, among them J1 Probes, J2 Probes, J3 eflashy32, U1 ESP32-WROOM-32D

Commit message: updates for v2
Parts:
- removed C13: 1uF, Capacitor_SMD:C_0603_1608Metric, symbol Device:C_Small
- removed J3: eflashy32, Connector_PinHeader_2.54mm:PinHeader_1x06_P2.54mm_Vertical, symbol Connector_Generic:Conn_01x06
- removed U1: ESP32-WROOM-32D, RF_Module:ESP32-WROOM-32, symbol RF_Module:ESP32-WROOM-32D
- added C2: 0.1u, Capacitor_SMD:C_0603_1608Metric, symbol Device:C_Small
- added C7: 10u, Capacitor_SMD:C_0805_2012Metric, symbol Device:C_Small
- added D7: PWR, LED_SMD:LED_0805_2012Metric, symbol Device:LED
- added R3, R4: 10k, Resistor_SMD:R_0402_1005Metric, symbol Device:R_Small
- added R9: 680, Resistor_SMD:R_0402_1005Metric, symbol Device:R_Small
- added SW1: RESET, Button_Switch_SMD:SW_Push_1P1T_XKB_TS-1187A, symbol Switch:SW_SPST
- added U1: ESP32-C3-MINI-1, Espressif:ESP32-C3-MINI-1, symbol Espressif:ESP32-C3-MINI-1
- C1: value 10uF -> 10u
Connections:
- net +3V3: now also R1.1, C2.2, C7.2, D7.2 (A), R3.1, R4.1, U1.3 (3V3); no longer C1.2, R1.2
- net EN: now also C1.2, R1.2, U1.8 (EN/CHIP_PU); no longer R1.1
- net GND: now also C2.1, C7.1, R9.2, SW1.2 (B), U1.1 (GND), U1.11 (GND), U1.14 (GND), U1.2 (GND), U1.36 (GND), U1.37 (GND), U1.38 (GND), U1.39 (GND), U1.40 (GND), U1.41 (GND), U1.42 (GND), U1.43 (GND), U1.44 (GND), U1.45 (GND), U1.46 (GND), U1.47 (GND), U1.48 (GND), U1.49 (GND), U1.50 (GND), U1.51 (GND), U1.52 (GND), U1.53 (GND)
- net GPIO0: now also SW1.1 (A), U1.23 (GPIO9)
- net PROBE_BUS: now also U1.20 (GPIO6)
- new net: D7.1 (K), R9.1
- new net: R4.2, U1.22 (GPIO8)
- new net: R3.2, U1.5 (GPIO2/ADC1_CH2)
- new net D+: U1.27 (GPIO19/USB_D+)
- new net D-: U1.26 (GPIO18/USB_D-)
- no-connect marks 28 -> 9
Other:
- note added: "C3 uses GPIO9 now"
- note removed: "(already has small bypass caps)"
- note removed: "34/35 are input only"
- note removed: "ESP32"
- note removed: "Programming"
- moved on the sheet: J1, J2, R2

Commit message: more v2 changes
Parts:
- removed J1, J2: Probes, TerminalBlock_Phoenix:TerminalBlock_Phoenix_MPT-0,5-12-2.54_1x12_P2.54mm_Horizontal, symbol Connector:Screw_Terminal_01x12
- added J1: T1, Connector_Phoenix_MC:PhoenixContact_MC_1,5_3-G-3.81_1x03_P3.81mm_Horizontal, symbol Connector:Screw_Terminal_01x03
- added J2: T2, Connector_Phoenix_MC:PhoenixContact_MC_1,5_3-G-3.81_1x03_P3.81mm_Horizontal, symbol Connector:Screw_Terminal_01x03
- added J4: T3, Connector_Phoenix_MC:PhoenixContact_MC_1,5_3-G-3.81_1x03_P3.81mm_Horizontal, symbol Connector:Screw_Terminal_01x03
- added J6: T4, Connector_Phoenix_MC:PhoenixContact_MC_1,5_3-G-3.81_1x03_P3.81mm_Horizontal, symbol Connector:Screw_Terminal_01x03
- H1, H2, H3, H4: now left out of the parts list
Connections:
- net +3V3: now also J1.1 (Pin_1), J2.1 (Pin_1), J4.1 (Pin_1), J6.1 (Pin_1)
- net GND: now also J1.3 (Pin_3), J2.3 (Pin_3), J4.3 (Pin_3), J6.3 (Pin_3)
- net PROBE_BUS: now also J1.2 (Pin_2), J2.2 (Pin_2), J4.2 (Pin_2), J6.2 (Pin_2)
- net GPIO0 renamed GPIO9
Other:
- note added: "Mechanical"
- note added: "Nets"
- note added: "Power LED"
- moved on the sheet: D7, H1, H2, H3, H4, R2, R3, R4, R9

Commit message: final touches and check
Other:
- note added: "C3 uses GPIO9"
- note removed: "C3 uses GPIO9 now"
- moved on the sheet: C1, C2, C7, D7, H1, H2, H3, H4, J1, J2, J4, J6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

Commit message: panel touchup, alternate pn
Parts:
- J1, J2, J6: LCSC Alt (none) -> C5188158
Changed lines of the file:
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@@
+			)
+		)
+		(property "LCSC Alt" "C5188158"
+			(at 222.25 34.29 0)
+			(effects
+				(font
+					(size 1.27 1.27)
+				)
+				(hide yes)
 			)
 		)
@@
 			)
 		)
+		(property "LCSC Alt" "C5188158"
+			(at 222.25 43.18 0)
+			(effects
+				(font
+					(size 1.27 1.27)
+				)
+				(hide yes)
+			)
+		)
 		(pin "1"
 		)
@@
 			(at 222.25 60.96 0)
 			(effects
+				(font
+					(size 1.27 1.27)
+				)
+				(hide yes)
+			)
+		)
+		(property "LCSC Alt" "C5188158"
+			(at 222.25 60.96 0)
+			(effects
