File: pcb/esptemp8c_panel2/esptemp8c_panel2.kicad_pcb (KiCad board)
At the start: 2 copper layers, 60 x 22.7 mm, 0 parts

Commit message: panel touchup, alternate pn
Other:
- board text added: "3V SIG GND"
Changed lines of the file:
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@@
 		(grid_origin 135.090983 102.730009)
 		(pcbplotparams
-			(layerselection 0x0001030_ffffffff)
+			(layerselection 0x00010f0_ffffffff)
 			(plot_on_all_layers_selection 0x0000000_00000000)
 			(disableapertmacros no)
@@
 			(usegerberattributes yes)
 			(usegerberadvancedattributes yes)
-			(creategerberjobfile yes)
+			(creategerberjobfile no)
 			(dashed_line_dash_ratio 12.000000)
 			(dashed_line_gap_ratio 3.000000)
@@
 		)
 	)
+	(gr_text "3V\nSIG\nGND"
+		(at 153.490983 86.930009 90)
+		(layer "F.SilkS")
+		(effects
+			(font
+				(size 2.2 2)
+				(thickness 0.3048)
+			)
+			(justify left top)
+		)
+	)
+	(gr_text "3V\nSIG\nGND"
+		(at 181.490983 86.930009 90)
+		(layer "F.SilkS")
+		(effects
+			(font
+				(size 2.2 2)
+				(thickness 0.3048)
+			)
+			(justify left top)
+		)
+	)
+	(gr_text "3V\nSIG\nGND"
+		(at 139.490983 86.930009 90)
+		(layer "F.SilkS")
+		(effects
+			(font
+				(size 2.2 2)
+				(thickness 0.3048)
+			)
+			(justify left top)
+		)
+	)
+	(gr_text "3V\nSIG\nGND"
+		(at 167.490983 86.930009 90)
+		(layer "F.SilkS")
+		(effects
+			(font
+				(size 2.2 2)
+				(thickness 0.3048)
+			)
+			(justify left top)
+		)
+	)
